File: pcb_smd_flightcontroller/pcb_smd_flightcontroller.kicad_sch (KiCad schematic)
At the start: 0 parts

Commit message: PCB STM32
Parts:
- added U1: STM32F411CEU6, aeasyeda:stm32f411, symbol easyedea:STM32F411CEU6
Connections:
- no-connect marks 0 -> 23
